Commit message: c30-rの干渉モデルを実装するためbedメッシュモデルの離れ小島を削除し、carrier側はbox形状として設定

File: Assets/c30-r_test_urdf.urdf (robot description, URDF)
Before this commit: robot c30-r, 5 links, 4 joints
Links:
- link bed_link: geometry collision mesh filename=package://c30-r_description/meshes/bed_removed.stl scale=0.001 0.001 0.001; visual mesh filename=package://c30-r_description/meshes/bed_removed.stl scale=0.001 0.001 0.001
- link body_link: geometry collision box size=3.25 1.5 0.8; visual mesh filename=package://c30-r_description/meshes/carrier.stl scale=0.001 0.001 0.001

Commit message: c30-rのurdfファイルを修正した-refineを作成しsceneへインポート

File: Assets/c30-r_test_urdf.urdf (robot description, URDF)
Before this commit: robot c30-r, 5 links, 4 joints
Links:
- added link left_front_wheel_link, mass 10; collision cylinder length=0.3 radius=0.25
- added link left_middle_wheel_link, mass 10; collision cylinder length=0.3 radius=0.25
- added link left_rear_wheel_link, mass 10; collision cylinder length=0.3 radius=0.25
- added link right_front_wheel_link, mass 10; collision cylinder length=0.3 radius=0.25
- added link right_middle_wheel_link, mass 10; collision cylinder length=0.3 radius=0.25
- added link right_rear_wheel_link, mass 10; collision cylinder length=0.3 radius=0.25
Joints:
- added joint left_front_wheel_joint: type continuous, parent base_link, child left_front_wheel_link, origin xyz=-0.1 0.6 0.1 rpy=-1.5707963267948966 0 0, axis 0 0 1
- added joint left_middle_wheel_joint: type continuous, parent base_link, child left_middle_wheel_link, origin xyz=-0.775 0.6 0.1 rpy=-1.5707963267948966 0 0, axis 0 0 1
- added joint left_rear_wheel_joint: type continuous, parent base_link, child left_rear_wheel_link, origin xyz=-1.45 0.6 0.1 rpy=-1.5707963267948966 0 0, axis 0 0 1
- added joint right_front_wheel_joint: type continuous, parent base_link, child right_front_wheel_link, origin xyz=-0.1 -0.6 0.1 rpy=-1.5707963267948966 0 0, axis 0 0 1
- added joint right_middle_wheel_joint: type continuous, parent base_link, child right_middle_wheel_link, origin xyz=-0.775 -0.6 0.1 rpy=-1.5707963267948966 0 0, axis 0 0 1
- added joint right_rear_wheel_joint: type continuous, parent base_link, child right_rear_wheel_link, origin xyz=-1.45 -0.6 0.1 rpy=-1.5707963267948966 0 0, axis 0 0 1
