Commit message: ic120とc30rのvesselにcontrollerのscriptを追加

File: Assets/c30-r_refine_urdf.urdf (robot description, URDF)
Before this commit: robot c30-r, 10 links, 9 joints
Links:
- link left_front_wheel_link: geometry collision cylinder length=0.3 radius=0.29
- link left_middle_wheel_link: geometry collision cylinder length=0.3 radius=0.29
- link left_rear_wheel_link: geometry collision cylinder length=0.3 radius=0.29
- link right_front_wheel_link: geometry collision cylinder length=0.3 radius=0.29
- link right_middle_wheel_link: geometry collision cylinder length=0.3 radius=0.29
- link right_rear_wheel_link: geometry collision cylinder length=0.3 radius=0.29
