Commit message: ショベルのモデルをフォーラムエイトが作成したものへ変更

File: Assets/Machines/zx120/zx120.urdf (robot description, URDF)
Before this commit: robot zx120, 14 links, 13 joints
Links:
- removed link link1
- removed link link10
- removed link link11
- removed link link12
- removed link link13
- removed link link2
- removed link link3
- removed link link4
- removed link link5
- removed link link6
- removed link link7
- removed link link8
- removed link link9
- removed link world
- added link arm_link, mass 0.03; collision mesh filename=package://zx120_description/meshes/zx120-arm.dae; visual mesh filename=package://zx120_description/meshes/zx120-arm.dae
- added link base_link
- added link body_link, mass 0.03; collision mesh filename=package://zx120_description/meshes/zx120-body.dae; visual mesh filename=package://zx120_description/meshes/zx120-body.dae
- added link boom_link, mass 0.03; collision mesh filename=package://zx120_description/meshes/zx120-boom.dae; visual mesh filename=package://zx120_description/meshes/zx120-boom.dae
- added link bucket_end_link, mass 1.0e-03; visual box size=0.001 0.001 0.001
- added link bucket_link, mass 0.03; collision mesh filename=package://zx120_description/meshes/zx120-bucket.dae; visual mesh filename=package://zx120_description/meshes/zx120-bucket.dae
- added link track_link, mass 10; collision mesh filename=package://zx120_description/meshes/zx120-crawler.dae; visual mesh filename=package://zx120_description/meshes/zx120-crawler.dae
Joints:
- removed joint fixed
- removed joint joint1
- removed joint joint10
- removed joint joint11
- removed joint joint12
- removed joint joint2
- removed joint joint3
- removed joint joint4
- removed joint joint5
- removed joint joint6
- removed joint joint7
- removed joint joint8
- removed joint joint9
- added joint arm_joint: type revolute, parent boom_link, child arm_link, origin xyz=0 0 4.6, axis 0 1 0, limit lower=0.523598775598 upper=2.65290046303 effort=1 velocity=0.5
- added joint base_joint: type fixed, parent base_link, child track_link
- added joint boom_joint: type revolute, parent body_link, child boom_link, origin xyz=0.14 -0.16443 0.424 rpy=0 1.57079632679 0, axis 0 1 0, limit lower=-1.2217304764 upper=0.767944870878 effort=500 velocity=6.159937255
- added joint bucket_end_joint: type revolute, parent bucket_link, child bucket_end_link, origin xyz=0 0 1.23 rpy=0 0.872664625997 0, axis 1 0 0, limit lower=-3.14 upper=3.14 effort=1 velocity=0.5
- added joint bucket_joint: type revolute, parent arm_link, child bucket_link, origin xyz=0 0 2.519, axis 0 1 0, limit lower=-0.575958653158 upper=2.49582083035 effort=1 velocity=0.5
- added joint swing_joint: type continuous, parent track_link, child body_link, origin xyz=0 0 1, axis 0 0 2
