Commit message: Newly made zx120 and ic120 models (from forum8) are imported

File: Assets/Machines/ic120/ic120.urdf (robot description, URDF)
Before this commit: robot ic120, 5 links, 4 joints
Links:
- link link1: mass 0.03 -> 1
- link link2: mass 0.03 -> 1
- link link3: mass 0.03 -> 1
- link link4: mass 0.03 -> 1
Joints:
- joint joint1: axis 1 0 0 -> 0 1 0; origin xyz=0 3.0153 0.94605 -> xyz=-3.015332 0 0.946052
- joint joint2: axis 1 0 0 -> 0 1 0; origin xyz=0 0.75792 0.73083 -> xyz=-0.75792 0 0.73083
- joint joint3: axis 0 1.4989 0.51788 -> -1.4989 0 0.51788

File: Assets/Machines/zx120/zx120.urdf (robot description, URDF)
Before this commit: robot zx120, 14 links, 13 joints
Joints:
- joint joint10: axis 0 0.021529 -2.207579 -> -0.021529 0 -2.207579
- joint joint11: axis 1 0 0 -> 0 1 0; origin xyz=0 -0.330489 -2.150643 -> xyz=0.330489 0 -2.150643
- joint joint12: axis 1 0 0 -> 0 1 0; origin xyz=0 0.182145 -0.315076 -> xyz=-0.182145 0 -0.315076
- joint joint2: axis 1 0 0 -> 0 1 0; origin xyz=-0.16443 -0.15433 0.31327 -> xyz=0.15433 -0.16443 0.31327
- joint joint3: axis 1 0 0 -> 0 1 0; origin xyz=0 -4.2241 1.7311 -> xyz=4.2241 0 1.7311
- joint joint4: axis 1 0 0 -> 0 1 0; origin xyz=0 -0.35383 -2.4712 -> xyz=0.35383 0 -2.4712
- joint joint5: axis 1 0 0 -> 0 1 0; origin xyz=-0.164428 -0.556105 0.032962 -> xyz=0.556105 -0.164428 0.032962
- joint joint6: axis 0 -0.802033 1.847495 -> 0.802033 0 1.847495
- joint joint7: axis 1 0 0 -> 0 1 0; origin xyz=0 -2.053030 1.991444 -> xyz=2.053030 0 1.991444
- joint joint8: axis 0 -2.36471 0 -> 2.36471 0 0
- joint joint9: axis 1 0 0 -> 0 1 0; origin xyz=0 -0.605825 -0.364793 -> xyz=0.605825 0 -0.364793

Commit message: フォーラムエイトが作成したic120のモデルを基にアセットを設定したオブジェクトを追加

File: Assets/Machines/ic120/ic120.urdf (robot description, URDF)
Before this commit: robot ic120, 5 links, 4 joints
Links:
- removed link link1
- removed link link2
- removed link link3
- removed link link4
- removed link world
- added link base_link, mass 1; collision mesh filename=package://meshes/ic120-body.dae; visual mesh filename=package://meshes/ic120-body.dae
- added link left_front_wheel_link, mass 10; collision cylinder length=0.1 radius=0.5
- added link left_middle_wheel_link, mass 10; collision cylinder length=0.1 radius=0.5
- added link left_rear_wheel_link, mass 10; collision cylinder length=0.1 radius=0.5
- added link right_front_wheel_link, mass 10; collision cylinder length=0.1 radius=0.5
- added link right_middle_wheel_link, mass 10; collision cylinder length=0.1 radius=0.5
- added link right_rear_wheel_link, mass 10; collision cylinder length=0.1 radius=0.5
- added link vessel_link, mass 1; collision mesh filename=package://meshes/ic120-bucket.dae; visual mesh filename=package://meshes/ic120-bucket.dae
Joints:
- removed joint fixed
- removed joint joint2
- removed joint joint3
- added joint left_front_wheel_joint: type continuous, parent base_link, child left_front_wheel_link, origin xyz=0.9 1 0.5 rpy=-1.5707963267948966 0 0, axis 0 0 1
- added joint left_middle_wheel_joint: type continuous, parent base_link, child left_middle_wheel_link, origin xyz=-0.6 1 0.5 rpy=-1.5707963267948966 0 0, axis 0 0 1
- added joint left_rear_wheel_joint: type continuous, parent base_link, child left_rear_wheel_link, origin xyz=-1.6 1 0.5 rpy=-1.5707963267948966 0 0, axis 0 0 1
- added joint right_front_wheel_joint: type continuous, parent base_link, child right_front_wheel_link, origin xyz=0.9 -1 0.5 rpy=-1.5707963267948966 0 0, axis 0 0 1
- added joint right_middle_wheel_joint: type continuous, parent base_link, child right_middle_wheel_link, origin xyz=-0.6 -1 0.5 rpy=-1.5707963267948966 0 0, axis 0 0 1
- added joint right_rear_wheel_joint: type continuous, parent base_link, child right_rear_wheel_link, origin xyz=-1.6 -1 0.5 rpy=-1.5707963267948966 0 0, axis 0 0 1
- joint joint1: child link2 -> vessel_link; parent link1 -> base_link
