Commit message: Sync ZX200 joint origins with zx200_ros2 URDF
zx200_ros2 main moved the working-range joint origins (PR #21, commit
3503f1b, plus the bucket_end_link origin from PR #19), so the Unity model
has to follow.

Assets/Prefab/zx200.prefab - per joint, the link transform and the
articulation parent anchor (Unity frame):
  boom_joint        (0.040187, 0.83669, 0.22767) -> (0.040187, 0.72492, 0.05467)
  arm_joint         (-0.010957, 2.9959, 4.7878)  -> (-0.010957, 3.00227, 4.83998)
  bucket_joint      (0.023546, 2.1809, 1.8954)   -> (0.023546, 2.17374, 1.91546)
  bucket_end_joint  (0, 1, 1.2)                  -> (0, 0.93856, 1.13012)
Frame rotations stay as they are for boom_joint/arm_joint, bucket_end_joint
returns to identity (rpy 0), both matching the URDF.

Two pre-existing mismatches are repaired along the way: a Unity
ArticulationBody takes its joint frame from the anchors, not from the child
transform, so leaving them behind would keep the old geometry alive in the
simulation.
  * boom_joint/arm_joint/bucket_joint parent anchor rotations were still the
    2023 URDF values (35/15/-20 deg) after 0bf9044 had updated only the link
    transforms and the euler hints;
  * bucket_joint's link frame was still -20 deg while its serialized euler
    hint already said -9.20083 deg, i.e. the value 0bf9044 intended.

Assets/Machines/zx200/zx200.urdf - the URDF this prefab was imported from -
still carried the 2023 values (rpy 35/15/-20 deg, bucket_end 1.2 0 1); it is
updated to the same origins so that URDF and prefab agree again.

Checked by parsing the prefab after the edit: for all four joints the link
transform, the parent anchor and the relation parent anchor rotation =
child pose * child anchor reproduce the URDF origin in the Unity frame
(-y, z, x), and the child anchors still match the axis frames that the URDF
importer generates.

File: Assets/Machines/zx200/zx200.urdf (robot description, URDF)
Before this commit: robot zx200, 12 links, 11 joints
Joints:
- joint arm_joint: origin xyz=4.7878 0.010957 2.9959 rpy=0 0.2617993878 0 -> xyz=4.83998 0.010957 3.00227 rpy=0 0.2961945914 0
- joint boom_joint: origin xyz=0.22767 -0.040187 0.83669 rpy=0 0.6108652382 0 -> xyz=0.05467 -0.040187 0.72492 rpy=0 0.5591284432 0
- joint bucket_end_joint: origin xyz=1.2 0 1 rpy=0 0 0 -> xyz=1.13012 0 0.93856 rpy=0 0 0
- joint bucket_joint: origin xyz=1.8954 -0.023546 2.1809 rpy=0 -0.3490658504 0 -> xyz=1.91546 -0.023546 2.17374 rpy=0 -0.1605847774 0
